File: USB_Power_Adapter/USB_Power_Adapter.brd (EAGLE design)
At the start: 29 x 17 mm, 6 parts

Commit message: Forced name U1
Parts:
- renumbered U$1 to U1
Changed lines of the file:
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@@
 </autorouter>
 <elements>
-<element name="U$1" library="ScottSilver" package="MICROUSB_THRU" value="MICROUSBMICROUSB_THRU" x="4.25" y="9"/>
+<element name="U1" library="ScottSilver" package="MICROUSB_THRU" value="MICROUSBMICROUSB_THRU" x="4.25" y="9"/>
 <element name="U$3" library="ScottSilver" package="SC189" value="SC189" x="8" y="9" smashed="yes" rot="R270"/>
 <element name="C1" library="resistor" package="C0805K" value="10uF" x="7.5" y="11.5" smashed="yes">
@@
 <signals>
 <signal name="N$1">
-<contactref element="U$1" pad="VCC"/>
+<contactref element="U1" pad="VCC"/>
 <contactref element="U$3" pad="1"/>
 <contactref element="U$3" pad="3"/>
@@
 </signal>
 <signal name="GND">
-<contactref element="U$1" pad="GND"/>
+<contactref element="U1" pad="GND"/>
 <contactref element="U$3" pad="2"/>
 <contactref element="C1" pad="2"/>

Commit message: Fixed junctions
Parts:
- removed U$3: SC189, ScottSilver:SC189
- added J1: MICROUSBMICROUSB_THRU, ScottSilver:MICROUSB_THRU
- U1: value MICROUSBMICROUSB_THRU -> SC189; device ScottSilver:MICROUSB_THRU -> ScottSilver:SC189
- moved U1 3.75 mm to (8.00, 9.00), turned to 270 degrees
Connections:
- net GND: now also J1.GND, U1.2; no longer U$3.2, U1.GND
- net LX: now also U1.5; no longer U$3.5
- net N$1: now also J1.VCC, U1.1, U1.3; no longer U$3.1, U$3.3, U1.VCC
- net N$3: now also U1.4; no longer U$3.4
Changed lines of the file:
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@@
 </autorouter>
 <elements>
-<element name="U1" library="ScottSilver" package="MICROUSB_THRU" value="MICROUSBMICROUSB_THRU" x="4.25" y="9"/>
-<element name="U$3" library="ScottSilver" package="SC189" value="SC189" x="8" y="9" smashed="yes" rot="R270"/>
+<element name="J1" library="ScottSilver" package="MICROUSB_THRU" value="MICROUSBMICROUSB_THRU" x="4.25" y="9"/>
+<element name="U1" library="ScottSilver" package="SC189" value="SC189" x="8" y="9" smashed="yes" rot="R270"/>
 <element name="C1" library="resistor" package="C0805K" value="10uF" x="7.5" y="11.5" smashed="yes">
 <attribute name="NAME" x="7.5" y="14" size="1.016" layer="25"/>
@@
 <signals>
 <signal name="N$1">
-<contactref element="U1" pad="VCC"/>
-<contactref element="U$3" pad="1"/>
-<contactref element="U$3" pad="3"/>
+<contactref element="J1" pad="VCC"/>
+<contactref element="U1" pad="1"/>
+<contactref element="U1" pad="3"/>
 <contactref element="C1" pad="1"/>
 <wire x1="4.25" y1="10.3" x2="6.5" y2="10.3" width="0.4064" layer="1"/>
@@
 </signal>
 <signal name="N$3">
-<contactref element="U$3" pad="4"/>
+<contactref element="U1" pad="4"/>
 <contactref element="C2" pad="1"/>
 <contactref element="L1" pad="2"/>
@@
 </signal>
 <signal name="LX">
-<contactref element="U$3" pad="5"/>
+<contactref element="U1" pad="5"/>
 <contactref element="L1" pad="1"/>
 <wire x1="9.25" y1="9.95" x2="10.25" y2="10.4" width="0.8128" layer="1"/>
@@
 </signal>
 <signal name="GND">
-<contactref element="U1" pad="GND"/>
-<contactref element="U$3" pad="2"/>
+<contactref element="J1" pad="GND"/>
+<contactref element="U1" pad="2"/>
 <contactref element="C1" pad="2"/>
 <contactref element="C2" pad="2"/>
